File: PCB Rev A/PowerSection.sch (KiCad schematic (older format))
At the start: 77 parts, among them J5 CONN_01X12, J6 CONN_01X04, J7 CONN_01X04, Q10 2N7000, Q11 N-Ch TO-263, Q12 N-Ch TO-263, Q13 N-Ch TO-263, Q14 N-Ch TO-263, Q15 2N7000, Q7 2N7000, Q8 2N7000, Q9 2N7000, U10 LM7805CT, U11 LM555CN, U12 IR2102, U13 LM555CN, U14 IR2102, U6 74HCT04, U9 74LS08

Commit message: Updated Rev A PCB
Parts:
- C27: symbol CP1_Small -> device1:CP1_Small
- C28, C29, C30, C31, C32, C33, C35, C36, C37, C38, C39, C40: symbol C -> device1:C
- C34, C41: symbol CP -> device1:CP
- D10, D11, D12, D13, D15, D19: symbol LED -> device1:LED
- D14, D16, D17, D22, D23, D24: symbol D -> device1:D
- D18, D25: symbol ZENER -> Q-Throttle-rescue:ZENER-RESCUE-Q-Throttle
- D20, D21, D26, D27: symbol D_Schottky -> device1:D_Schottky
- J5: symbol CONN_01X12 -> Q-Throttle-rescue:CONN_01X12-RESCUE-Q-Throttle
- J6, J7: symbol CONN_01X04 -> Q-Throttle-rescue:CONN_01X04-RESCUE-Q-Throttle
- Q10, Q15, Q7, Q8, Q9: symbol Q_NMOS_SGD -> device1:Q_NMOS_SGD
- Q11, Q12, Q13, Q14: symbol Q_NMOS_GDS -> device1:Q_NMOS_GDS
- R32, R33, R34, R35, R36, R37, R38, R39, R40, R41, R42, R43, R44, R45, R46, R47, R48, R49, R50, R51, R52, R53, R54, R56, R57: symbol R -> device1:R
- U10: symbol LM7805CT -> Q-Throttle-rescue:LM7805CT-RESCUE-Q-Throttle
- U11, U13: symbol LM555CN -> lm555cn:LM555CN
- U12, U14: symbol IR2102 -> Q-Throttle-rescue:IR2102-RESCUE-Q-Throttle
- U6: symbol 74HCT04 -> Q-Throttle-rescue:74HCT04-RESCUE-Q-Throttle
- U9: symbol 74LS08 -> Q-Throttle-rescue:74LS08-RESCUE-Q-Throttle
