File: PCB Rev A/Q-Throttle.kicad_pcb (KiCad board)
At the start: 2 copper layers, 167.6 x 127 mm, 177 parts, among them J1 CONN_01X08, J2 RJ-11, J3 CONN_01X05, J4 CONN_01X06, J5 CONN_01X12, J6 CONN_01X04, J7 CONN_01X04, Q1 2N7000, Q10 2N7000, Q11 N-Ch TO-263, Q12 N-Ch TO-263, Q13 N-Ch TO-263, Q14 N-Ch TO-263, Q15 2N7000, Q2 2N7000, Q3 Q_PMOS_GDS, Q4 2N7000, Q5 2N7000, Q6 2N7000, Q7 2N7000, Q8 2N7000, Q9 2N7000, SW1 SW_PUSH, U1 SP3485CN, U10 LM7805CT, U11 LM555CN, U12 IR2102, U13 LM555CN, U14 IR2102, U15 LM78Lxx, U17 XBee_S1, U2 LM6132A, U3 74LS125_(3V3), U4 LM2677-12, U5 MB85RC256V, U6 74HCT04, U7 LM358, U8 PIC16(L)F1938-I/SP, U9 74LS08

Commit message: Updated Rev A PCB
Parts:
- C24, C4: footprint Capacitors_ThroughHole:C_Radial_D10_L20_P7.5 -> Capacitors_THT:CP_Radial_D17.0mm_P7.50mm
- L2: footprint Choke_Toroid_ThroughHole:Choke_Toroid_8x16mm_Vertical -> Choke_Toroid_ThroughHole:Choke_Toroid_12x24mm_Vertical
- moved C4 9.92 mm to (61.0, 118.1), turned to 180 degrees
- moved R22 8.25 mm to (148.6, 152.4)
- moved C5 5.08 mm to (68.6, 123.2)
- moved D7 4.44 mm to (127.0, 142.9)
- moved C24 4.07 mm to (149.9, 139.7)
- moved Q2 3.86 mm to (121.9, 148.6)
- moved C7 3.81 mm to (74.9, 123.2)
- moved L2 3.24 mm to (132.1, 129.5)
- moved C8 2.54 mm to (81.3, 123.2)
- moved R15 2.54 mm to (118.1, 148.0)
- moved R16 1.91 mm to (121.9, 142.2), turned to 270 degrees
- moved C11 1.27 mm to (87.6, 123.2)
Routing:
- net GND: track 1018.9 -> 983.0 mm
- net M+: track 175.1 -> 198.4 mm
- net +15V: track 409.4 -> 419.3 mm
- net +24V: track 80.9 -> 87.6 mm
- net Net-(D7-Pad1): track 25.3 -> 29.5 mm
- net Net-(Q2-Pad2): track 8.81 -> 4.74 mm
- net Net-(Q2-Pad3): track 4.67 -> 2.46 mm
- net Net-(Q3-Pad1): track 16.0 -> 14.8 mm
Other:
- board text added: "Model Railroad Throttle Rev: A DMFE 2017"
- board text removed: "Model Railroad Throttle Rev: nc DMFE 2017"
